Commit message: manipulation package added

File: ws_husky_ur5/husky_ur5_description/urdf/kinect.xacro (robot description, xacro)
@@ -5,5 +5,5 @@
   <joint name="camera_joint" type="fixed">
     <axis xyz="1 0 0" />
-    <origin xyz="0.042 0.22 0.05" rpy="0 0 ${PI/2}"/> <!-- -40 degress-->
+    <origin xyz="-0.1 0.25 0.05" rpy="0 0 ${PI/4}"/> <!-- -40 degress-->
     <parent link="top_plate_link"/>
     <child link="kinect2_link"/>
@@ -55,5 +55,5 @@
     </link>
     <gazebo reference="kinect2_link">
-    <material>Gazebo/Black</material>
+    <material>Gazebo/White</material>
     <mu1 value= "0.3" />
     <mu2 value= "0.3" />

Commit message: Update kinect.xacro

File: ws_husky_ur5/husky_ur5_description/urdf/kinect.xacro (robot description, xacro)
@@ -32,5 +32,6 @@
       <origin xyz="-0.12 0.125 -0.04" rpy="0 0 -${PI/2}"/>
       <geometry>
-	<mesh filename="package://abb_barrett_description/meshes/kinect.STL" scale="0.001 0.001 0.001"/>/>
+	  <box size="0.05 0.05 0.1"/>
+	<!--mesh filename="package://abb_barrett_description/meshes/kinect.STL" scale="0.001 0.001 0.001"/>/-->
       </geometry>
     </collision>
@@ -38,5 +39,6 @@
       <origin xyz="-0.12 0.125 -0.04" rpy="0 0 -${PI/2}"/>
       <geometry>
-		<mesh filename="package://abb_barrett_description/meshes/kinect.STL" scale="0.001 0.001 0.001"/>/>
+		<box size="0.05 0.05 0.1"/>
+	      <!--mesh filename="package://abb_barrett_description/meshes/kinect.STL" scale="0.001 0.001 0.001"/>/-->
       </geometry>
       <material name="red"/>

Commit message: Added ABB stl files

File: ws_husky_ur5/husky_ur5_description/urdf/kinect.xacro (robot description, xacro)
@@ -32,6 +32,6 @@
       <origin xyz="-0.12 0.125 -0.04" rpy="0 0 -${PI/2}"/>
       <geometry>
-	  <box size="0.05 0.05 0.1"/>
-	<!--mesh filename="package://abb_barrett_description/meshes/kinect.STL" scale="0.001 0.001 0.001"/>/-->
+<!-- 	  <box size="0.05 0.05 0.1"/> -->
+	<mesh filename="package://abb_barrett_description/meshes/kinect.STL" scale="0.001 0.001 0.001"/>/
       </geometry>
     </collision>
@@ -39,6 +39,6 @@
       <origin xyz="-0.12 0.125 -0.04" rpy="0 0 -${PI/2}"/>
       <geometry>
-		<box size="0.05 0.05 0.1"/>
-	      <!--mesh filename="package://abb_barrett_description/meshes/kinect.STL" scale="0.001 0.001 0.001"/>/-->
+<!-- 		<box size="0.05 0.05 0.1"/> -->
+	 <mesh filename="package://abb_barrett_description/meshes/kinect.STL" scale="0.001 0.001 0.001"/>/
       </geometry>
       <material name="red"/>
