Commit message: updated

File: bhand/barrett_hand/urdf/barrett.xacro (robot description, xacro)
@@ -1,18 +1,18 @@
 <?xml version="1.0"?>
-<robot xmlns:xacro="http://www.ros.org/wiki/xacro">
-<property name="dist_joint_offset" value="0.75" />
-<property name="dist_joint_multiplier" value="0.3" />
-<property name="finger_stop_kd"             value="1.0" />
-<property name="finger_stop_kp"             value="10000000.0" />
-<property name="finger_fudge_factor"        value="1.0" />
-<property name="finger_kp"                  value="0.0" />
-<property name="finger_kd"                  value="0.0" />
-<property name="finger_fm"                  value="0.0" />
-<property name="finger_tip_kp"              value="0.0" />
-<property name="finger_tip_kd"              value="0.0" />
-<property name="finger_tip_fm"              value="0.0" />
-<property name="finger_tip_mu"              value="1500.0" />
-<property name="finger_mu"                  value="1500.0" />
-<property name="dist_joint_multiplier" value="0.3" />
+<robot xmlns:xacro="http://ros.org/wiki/xacro">
+<xacro:property name="dist_joint_offset" value="0.75" />
+<xacro:property name="dist_joint_multiplier" value="0.3" />
+<xacro:property name="finger_stop_kd"             value="1.0" />
+<xacro:property name="finger_stop_kp"             value="10000000.0" />
+<xacro:property name="finger_fudge_factor"        value="1.0" />
+<xacro:property name="finger_kp"                  value="0.0" />
+<xacro:property name="finger_kd"                  value="0.0" />
+<xacro:property name="finger_fm"                  value="0.0" />
+<xacro:property name="finger_tip_kp"              value="0.0" />
+<xacro:property name="finger_tip_kd"              value="0.0" />
+<xacro:property name="finger_tip_fm"              value="0.0" />
+<xacro:property name="finger_tip_mu"              value="1500.0" />
+<xacro:property name="finger_mu"                  value="1500.0" />
+<xacro:property name="dist_joint_multiplier" value="0.3" />
    <link name="barrett_base_link">
     <inertial>

File: ws_husky_ur5/husky_ur5_description/urdf/husky_ur5.urdf (robot description, URDF)
Before this commit: robot husky_ur5, 36 links, 35 joints
Links:
- removed link top_plate_front_link
- removed link top_plate_rear_link
- added link kinect2_depth_optical_frame
- added link kinect2_link, mass 1e-5; collision mesh filename=package://abb_barrett_description/meshes/kinect.STL scale=0.001 0.001 0.001; visual mesh filename=package://abb_barrett_description/meshes/kinect.STL scale=0.001 0.001 0.001
- added link kinect2_rgb_optical_frame
- added link offset_optical_frame
Joints:
- removed joint top_plate_front_joint
- removed joint top_plate_rear_joint
- added joint camera1_joint: type fixed, parent kinect2_link, child kinect2_depth_optical_frame, origin xyz=0.0 -0.0 0 rpy=-1.57079632679 0 -1.57079632679, axis 1 0 0
- added joint camera2_joint: type fixed, parent kinect2_link, child kinect2_rgb_optical_frame, origin xyz=0.0 -0.0 0 rpy= -1.57079632679 0 -1.57079632679, axis 1 0 0
- added joint camera_joint: type fixed, parent top_plate_link, child kinect2_link, origin xyz=-0.1 0.25 0.05 rpy=0 0 0.785398163397, axis 1 0 0
- added joint offset_camera_joint: type fixed, parent kinect2_link, child offset_optical_frame, origin xyz=0 0 -0.05 rpy=-1.57079632679 0 -1.57079632679, axis 1 0 0
- joint world-base_link-fixed: origin xyz=0 0 0.33 rpy=0 0 0 -> xyz=0 0 0.15 rpy=0 0 0

File: ws_husky_ur5/husky_ur5_description/urdf/kinect.xacro (robot description, xacro)
@@ -5,5 +5,5 @@
   <joint name="camera_joint" type="fixed">
     <axis xyz="1 0 0" />
-    <origin xyz="-0.1 0.25 0.05" rpy="0 0 ${PI/4}"/> <!-- -40 degress-->
+    <origin xyz="0.32 0 -0.05" rpy="0 0 0"/> <!-- -40 degress-->
     <parent link="top_plate_link"/>
     <child link="kinect2_link"/>

Commit message: grasp hack working

File: bhand/barrett_hand/urdf/barrett.xacro (robot description, xacro)
@@ -76,5 +76,5 @@
     </collision>
   </link>
-  <!--joint name="finger_1_prox_joint" type="revolute">
+  <joint name="finger_1_prox_joint" type="revolute">
     <origin xyz="0.025 0 0.0415" rpy="0 2.7051E-17 -1.5708" />
     <parent link="barrett_base_link" />
@@ -83,12 +83,4 @@
     <limit lower="0.0" upper="3.141" effort="10000" velocity="0.2" />
    <dynamics damping="10.0" friction="10.0" />
-  </joint-->
-  <joint name="finger_1_prox_joint" type="revolute">
-    <origin xyz="0.025 0 0.0415" rpy="0 2.7051E-17 3.67" />
-    <parent link="barrett_base_link" />
-    <child link="finger_1_prox_link" />
-    <axis xyz="0 0 -1" />
-    <limit lower="0.0" upper="3.141" effort="10000" velocity="0.2" />
-   <dynamics damping="10.0" friction="10.0" />
   </joint>
   <link
@@ -123,5 +115,5 @@
     </collision>
   </link>
-  <!--joint
+  <joint
     name="finger_1_med_joint"
     type="revolute">
@@ -132,14 +124,4 @@
     <limit lower="0" upper="2.44" effort="10000" velocity="0.2" />
    <dynamics damping="10.0" friction="10.0" />
-  </joint-->
-  <joint
-    name="finger_1_med_joint"
-    type="revolute">
-    <origin xyz="-0.05 0 0.0339" rpy="-1.5708 1.5708 0" />
-    <parent link="finger_1_prox_link" />
-    <child link="finger_1_med_link" />
-    <axis xyz="0 0 1" />
-    <limit lower="0" upper="2.44" effort="10000" velocity="0.2" />
-   <dynamics damping="10.0" friction="10.0" />
   </joint>
   <link
@@ -198,5 +180,5 @@
     </collision>
   </link>
-  <!--joint name="finger_2_prox_joint" type="revolute">
+  <joint name="finger_2_prox_joint" type="revolute">
     <origin xyz="-0.025 0 0.0415" rpy="0 2.7051E-17 -1.5708" />
     <parent link="barrett_base_link" />
@@ -205,12 +187,4 @@
     <limit lower="0" upper="3.141" effort="10000"  velocity="0.2" />
    <dynamics damping="10.0" friction="10.0" />
-  </joint-->
-  <joint name="finger_2_prox_joint" type="revolute">
-    <origin xyz="-0.025 0 0.0415" rpy="0 2.7051E-17 -0.52" />
-    <parent link="barrett_base_link" />
-    <child link="finger_2_prox_link" />
-    <axis xyz="0 0 1" />
-    <limit lower="0" upper="3.141" effort="10000"  velocity="0.2" />
-   <dynamics damping="10.0" friction="10.0" />
   </joint>
   <link
@@ -245,18 +219,8 @@
     </collision>
   </link>
-  <!--joint
+  <joint
     name="finger_2_med_joint"
     type="revolute">
     <origin xyz="-0.05 0 0.0339" rpy="-1.5708 -8.8281E-17 0" />
-    <parent link="finger_2_prox_link" />
-    <child link="finger_2_med_link" />
-    <axis xyz="0 0 1" />
-    <limit lower="0.0" upper="2.44" effort="10000" velocity="0.2" />
-   <dynamics damping="10.0" friction="10.0" />
-  </joint-->
-  <joint
-    name="finger_2_med_joint"
-    type="revolute">
-    <origin xyz="-0.05 0 0.0339" rpy="-1.5708 1.5708 0" />
     <parent link="finger_2_prox_link" />
     <child link="finger_2_med_link" />
@@ -342,5 +306,5 @@
     </collision>
   </link>
-  <!--joint
+  <joint
     name="finger_3_med_joint"
     type="revolute">
@@ -348,23 +312,4 @@
       xyz="0 -0.05 0.0754"
       rpy="-1.5708 6.123E-17 1.5708" />
-    <parent
-      link="barrett_base_link" />
-    <child
-      link="finger_3_med_link" />
-    <axis
-      xyz="0 0 1" />
-    <limit
-      lower="0.0"
-      upper="2.44"
-      effort="10000"
-      velocity="0.2" />
-   <dynamics damping="10.0" friction="10.0" />
-  </joint-->
-  <joint
-    name="finger_3_med_joint"
-    type="revolute">
-    <origin
-      xyz="0 -0.05 0.0754"
-      rpy="-1.5708 1.5708 1.5708" />
     <parent
       link="barrett_base_link" />
@@ -549,6 +494,7 @@
   <gazebo reference="finger_1_dist_link">
      <turnGravityOff>true</turnGravityOff>
-      <mu1 value="${finger_mu}" />
-      <mu2 value="${finger_mu}" />
+     <implicitSpringDamper>1</implicitSpringDamper>
+      <mu1 value="${finger_tip_mu}" />
+      <mu2 value="${finger_tip_mu}" />
       <kp value="1000000.0" />
       <kd value="1.0" />
@@ -581,4 +527,14 @@
   <!-- finger_2_dist_link -->
   <gazebo reference="finger_2_dist_link">
+  <implicitSpringDamper>1</implicitSpringDamper>
+     <turnGravityOff>true</turnGravityOff>
+      <mu1 value="${finger_tip_mu}" />
+      <mu2 value="${finger_tip_mu}" />
+      <kp value="1000000.0" />
+      <kd value="1.0" />
+    <material>Gazebo/Grey</material>
+  </gazebo>
+  <!-- finger_3_med_link -->
+  <gazebo reference="finger_3_med_link">
      <turnGravityOff>true</turnGravityOff>
       <mu1 value="${finger_mu}" />
@@ -586,20 +542,12 @@
       <kp value="1000000.0" />
       <kd value="1.0" />
-    <material>Gazebo/Grey</material>
-  </gazebo>
-  <!-- finger_3_med_link -->
-  <gazebo reference="finger_3_med_link">
-     <turnGravityOff>true</turnGravityOff>
-      <mu1 value="${finger_mu}" />
-      <mu2 value="${finger_mu}" />
-      <kp value="1000000.0" />
-      <kd value="1.0" />
     <material>Gazebo/Black</material>
   </gazebo>
   <!-- finger_3_dist_link -->
   <gazebo reference="finger_3_dist_link">
-     <turnGravityOff>true</turnGravityOff>
-      <mu1 value="${finger_mu}" />
-      <mu2 value="${finger_mu}" />
+  <implicitSpringDamper>1</implicitSpringDamper>
+     <turnGravityOff>true</turnGravityOff>
+      <mu1 value="${finger_tip_mu}" />
+      <mu2 value="${finger_tip_mu}" />
       <kp value="1000000.0" />
       <kd value="1.0" />
@@ -620,11 +568,12 @@
       <gripper name="barrett_grasp_hack">
         <grasp_check>
-          <attach_steps>20</attach_steps>
-          <detach_steps>40</detach_steps>
-          <min_contact_count>2</min_contact_count>
+          <attach_steps>4</attach_steps>
+          <detach_steps>2</detach_steps>
+          <min_contact_count>1</min_contact_count>
         </grasp_check>
-        <gripper_link>finger_1_prox_link</gripper_link>
-        <gripper_link>finger_2_prox_link</gripper_link>
+        <gripper_link>finger_1_dist_link</gripper_link>
+        <gripper_link>finger_2_dist_link</gripper_link>
         <palm_link>barrett_base_link</palm_link>
+        <contact_topic>__default_topic__</contact_topic>
       </gripper>
     </gazebo>

File: ws_husky_ur5/husky_ur5_description/urdf/husky_ur5.urdf.xacro (robot description, xacro)
@@ -2,27 +2,20 @@
 <robot name="husky_ur5" xmlns:xacro="http://ros.org/wiki/xacro">
   <xacro:property name="PI" value="3.1415926535897931"/>
-  <xacro:include filename="$(find ur_description)/urdf/ur5.urdf.xacro"/>
+  <xacro:include filename="$(find husky_ur5_description)/urdf/abb_macro2.xacro"/>
   <xacro:include filename="$(find husky_description)/urdf/husky.urdf.xacro"/>
-  <!--xacro:include filename="$(find ur_description)/urdf/common.gazebo.xacro" /-->
-  <xacro:include filename="$(find barrett_hand)/urdf/barrett.xacro" />
-  <xacro:include filename="$(find husky_ur5_description)/urdf/kinect.xacro" />
-  <xacro:ur5_robot prefix="ur" joint_limited=" False"/>
-  <!-- Fix robot to Gazebo world-->
-  <link name="world"/>
-  <joint name="world-base_link-fixed" type="fixed">
-  	<origin xyz="0 0 0.15" rpy="0 0 0"/>
-    <parent link="world"/>
-    <child link="base_link"/>
-  </joint> >
-  <joint name="husky_ur5_joint" type="fixed">
+  <xacro:include filename="$(find barrett_hand)/urdf/barrett.xacro"/>
+  <xacro:include filename="$(find husky_ur5_description)/urdf/kinect.xacro"/>
+  <!-- Fix robot to Gazebo world
+  <link name="world"/>-->
+  <joint name="husky_abb" type="fixed">
+  	<origin xyz="0.3 0 0.25" rpy="0 0 0"/>
+    <parent link="base_link"/>
+    <child link="abb2_base_link"/>
+  </joint>
+    <xacro:abb2 prefix="abb2_"/>
+  <joint name="abb_barrett_joint" type="fixed">
     <axis xyz="0 1 0" />
-    <origin xyz="0.25 0 0.015" rpy="0 0 0"/>
-    <parent link="top_plate_link"/>
-    <child link="urbase_link"/>
-  </joint>
-  <joint name="ur5_robotiq_joint" type="fixed">
-    <axis xyz="0 1 0" />
-    <origin xyz="0.0015 0 0" rpy="0 1.570795  0"/>
-    <parent link="uree_link"/>
+    <origin xyz="0.0015 0 0" rpy="1.57 0 1.57"/>
+    <parent link="abb2_link_6"/>
     <child link="barrett_base_link"/>
   </joint>

Commit message: grasp hack definetly working

File: bhand/barrett_hand/urdf/barrett.xacro (robot description, xacro)
@@ -566,13 +566,19 @@
       </plugin>
       <!-- a formal implementation of grasp hack in gazebo with fixed joint -->
-      <gripper name="barrett_grasp_hack">
+      <gripper name="barrett_hand">
         <grasp_check>
-          <attach_steps>50</attach_steps>
-          <detach_steps>2</detach_steps>
+          <attach_steps>4</attach_steps>
+          <detach_steps>20</detach_steps>
           <min_contact_count>1</min_contact_count>
         </grasp_check>
         <gripper_link>finger_3_dist_link</gripper_link>
+        <gripper_link>finger_1_prox_link</gripper_link>
+        <gripper_link>finger_2_prox_link</gripper_link>
+        <gripper_link>finger_1_dist_link</gripper_link>
         <gripper_link>finger_2_dist_link</gripper_link>
-        <palm_link>palm_frame</palm_link>
+        <gripper_link>finger_1_med_link</gripper_link>
+        <gripper_link>finger_2_med_link</gripper_link>
+        <gripper_link>finger_3_med_link</gripper_link>
+        <palm_link>barrett_base_link</palm_link>
         <contact_topic>__default_topic__</contact_topic>
       </gripper>

File: ws_husky_ur5/husky_ur5_description/urdf/husky_ur5.urdf.xacro (robot description, xacro)
@@ -9,5 +9,5 @@
   <link name="world"/>-->
   <joint name="husky_abb" type="fixed">
-  	<origin xyz="0.3 0 0.25" rpy="0 0 0"/>
+  	<origin xyz="0.3 0 0.253" rpy="0 0 0"/>
     <parent link="base_link"/>
     <child link="abb2_base_link"/>
@@ -16,5 +16,5 @@
   <joint name="abb_barrett_joint" type="fixed">
     <axis xyz="0 1 0" />
-    <origin xyz="0.0015 0 0" rpy="1.57 0 1.57"/>
+    <origin xyz="0.0025 0 0" rpy="1.57 0 1.57"/>
     <parent link="abb2_link_6"/>
     <child link="barrett_base_link"/>

Commit message: fixed abb_barrett_description depenencies

File: bhand/barrett_hand/urdf/barrett.xacro (robot description, xacro)
@@ -26,5 +26,5 @@
         rpy="0 0 0" />
       <geometry>
-        <mesh filename="package://abb_barrett_description/meshes/base_link.STL" />
+        <mesh filename="package://barrett_hand/meshes/base_link.STL" />
       </geometry>
       <material name="">
@@ -35,5 +35,5 @@
       <origin xyz="0 0 0" rpy="0 0 0" />
       <geometry>
-        <mesh filename="package://abb_barrett_description/meshes/base_link.STL" />
+        <mesh filename="package://barrett_hand/meshes/base_link.STL" />
       </geometry>
     </collision>
@@ -58,5 +58,5 @@
       <geometry>
         <mesh
-          filename="package://abb_barrett_description/meshes/finger_1_prox_link.STL" />
+          filename="package://barrett_hand/meshes/finger_1_prox_link.STL" />
       </geometry>
       <material
@@ -72,5 +72,5 @@
       <geometry>
         <mesh
-          filename="package://abb_barrett_description/meshes/finger_1_prox_link.STL" />
+          filename="package://barrett_hand/meshes/finger_1_prox_link.STL" />
       </geometry>
     </collision>
@@ -97,5 +97,5 @@
       <geometry>
         <mesh
-          filename="package://abb_barrett_description/meshes/finger_1_med_link.STL" />
+          filename="package://barrett_hand/meshes/finger_1_med_link.STL" />
       </geometry>
       <material
@@ -111,5 +111,5 @@
       <geometry>
         <mesh
-          filename="package://abb_barrett_description/meshes/finger_1_med_link.STL" />
+          filename="package://barrett_hand/meshes/finger_1_med_link.STL" />
       </geometry>
     </collision>
@@ -135,5 +135,5 @@
       <origin xyz="0 0 0" rpy="3.14159265359 0 -0.73" />
       <geometry>
-        <mesh filename="package://abb_barrett_description/meshes/finger_1_dist_link.STL" />
+        <mesh filename="package://barrett_hand/meshes/finger_1_dist_link.STL" />
       </geometry>
       <material name="">
@@ -144,5 +144,5 @@
       <origin xyz="0 0 0" rpy="3.14159265359 0 -0.73" />
       <geometry>
-        <mesh filename="package://abb_barrett_description/meshes/finger_1_dist_link.STL" />
+        <mesh filename="package://barrett_hand/meshes/finger_1_dist_link.STL" />
       </geometry>
     </collision>
@@ -167,5 +167,5 @@
       <origin xyz="0 0 0" rpy="0 0 0" />
       <geometry>
-        <mesh filename="package://abb_barrett_description/meshes/finger_2_prox_link.STL" />
+        <mesh filename="package://barrett_hand/meshes/finger_2_prox_link.STL" />
       </geometry>
       <material name="">
@@ -176,5 +176,5 @@
       <origin xyz="0 0 0" rpy="0 0 0" />
       <geometry>
-        <mesh filename="package://abb_barrett_description/meshes/finger_2_prox_link.STL" />
+        <mesh filename="package://barrett_hand/meshes/finger_2_prox_link.STL" />
       </geometry>
     </collision>
@@ -201,5 +201,5 @@
       <geometry>
         <mesh
-          filename="package://abb_barrett_description/meshes/finger_2_med_link.STL" />
+          filename="package://barrett_hand/meshes/finger_2_med_link.STL" />
       </geometry>
       <material
@@ -215,5 +215,5 @@
       <geometry>
         <mesh
-          filename="package://abb_barrett_description/meshes/finger_2_med_link.STL" />
+          filename="package://barrett_hand/meshes/finger_2_med_link.STL" />
       </geometry>
     </collision>
@@ -239,5 +239,5 @@
       <origin xyz="0 0 0" rpy="3.14159265359 0 -0.73" />
       <geometry>
-        <mesh filename="package://abb_barrett_description/meshes/finger_2_dist_link.STL" />
+        <mesh filename="package://barrett_hand/meshes/finger_2_dist_link.STL" />
       </geometry>
       <material name="">
@@ -251,5 +251,5 @@
       <geometry>
         <mesh
-          filename="package://abb_barrett_description/meshes/finger_2_dist_link.STL" />
+          filename="package://barrett_hand/meshes/finger_2_dist_link.STL" />
       </geometry>
     </collision>
@@ -288,5 +288,5 @@
       <geometry>
         <mesh
-          filename="package://abb_barrett_description/meshes/finger_3_med_link.STL" />
+          filename="package://barrett_hand/meshes/finger_3_med_link.STL" />
       </geometry>
       <material
@@ -302,5 +302,5 @@
       <geometry>
         <mesh
-          filename="package://abb_barrett_description/meshes/finger_3_med_link.STL" />
+          filename="package://barrett_hand/meshes/finger_3_med_link.STL" />
       </geometry>
     </collision>
@@ -338,5 +338,5 @@
       <geometry>
         <mesh
-          filename="package://abb_barrett_description/meshes/finger_3_dist_link.STL" />
+          filename="package://barrett_hand/meshes/finger_3_dist_link.STL" />
       </geometry>
       <material
@@ -352,5 +352,5 @@
       <geometry>
         <mesh
-          filename="package://abb_barrett_description/meshes/finger_3_dist_link.STL" />
+          filename="package://barrett_hand/meshes/finger_3_dist_link.STL" />
       </geometry>
     </collision>

File: ws_husky_ur5/husky_ur5_description/urdf/kinect.xacro (robot description, xacro)
@@ -33,5 +33,5 @@
       <geometry>
 <!-- 	  <box size="0.05 0.05 0.1"/> -->
-	<mesh filename="package://abb_barrett_description/meshes/kinect.STL" scale="0.001 0.001 0.001"/>/
+	<mesh filename="package://husky_ur5_description/meshes/kinect/kinect.STL" scale="0.001 0.001 0.001"/>/
       </geometry>
     </collision>
@@ -40,5 +40,5 @@
       <geometry>
 <!-- 		<box size="0.05 0.05 0.1"/> -->
-	 <mesh filename="package://abb_barrett_description/meshes/kinect.STL" scale="0.001 0.001 0.001"/>/
+	 <mesh filename="package://husky_ur5_description/meshes/kinect/kinect.STL" scale="0.001 0.001 0.001"/>/
       </geometry>
       <material name="red"/>
