Commit message: Add files via upload

File: ws_husky_abb/husky_abb_description/urdf/abb_macro1.xacro (robot description, xacro)
@@ -17,5 +17,5 @@
         <xacro:material_abb_orange />
       </visual>
-      <collision>
+      <!--<collision>
         <origin xyz="0 0 0" rpy="0 0 0"/>
         <geometry>
@@ -23,5 +23,5 @@
         </geometry>
         <xacro:material_abb_yellow />
-      </collision>
+      </collision>-->
     </link>
     <link name="${prefix}link_1">
@@ -38,5 +38,5 @@
         <xacro:material_abb_orange />
       </visual>
-      <collision>
+      <!--<collision>
         <origin xyz="0 0 0" rpy="0 0 0"/>
         <geometry>
@@ -44,5 +44,5 @@
         </geometry>
         <xacro:material_abb_yellow />
-      </collision>
+      </collision>-->
     </link>
     <link name="${prefix}link_2">
@@ -59,5 +59,5 @@
         <xacro:material_abb_orange />
       </visual>
-      <collision>
+      <!--<collision>
         <origin xyz="0 0 0" rpy="0 0 0"/>
         <geometry>
@@ -65,5 +65,5 @@
         </geometry>
         <xacro:material_abb_yellow />
-      </collision>
+      </collision>-->
     </link>
     <link name="${prefix}link_3">
@@ -80,5 +80,5 @@
         <xacro:material_abb_orange />
       </visual>
-      <collision>
+      <!--<collision>
         <origin xyz="0 0 0" rpy="0 0 0"/>
         <geometry>
@@ -86,5 +86,5 @@
         </geometry>
         <xacro:material_abb_yellow />
-      </collision>
+      </collision>-->
     </link>
     <link name="${prefix}link_4">
@@ -101,5 +101,5 @@
         <xacro:material_abb_orange />
       </visual>
-      <collision>
+      <!--<collision>
         <origin xyz="0 0 0" rpy="0 0 0"/>
         <geometry>
@@ -107,5 +107,5 @@
         </geometry>
         <xacro:material_abb_yellow />
-      </collision>
+      </collision>-->
     </link>
     <link name="${prefix}link_5">
@@ -122,5 +122,5 @@
         <xacro:material_abb_orange />
       </visual>
-      <collision>
+      <!--<collision>
         <origin xyz="0 0 0" rpy="0 0 0"/>
         <geometry>
@@ -128,5 +128,5 @@
         </geometry>
         <xacro:material_abb_yellow />
-      </collision>
+      </collision>-->
     </link>
     <link name="${prefix}link_6">
@@ -143,5 +143,5 @@
         <xacro:material_abb_black />
       </visual>
-      <collision>
+      <!--<collision>
         <origin xyz="0 0 0" rpy="0 0 0"/>
         <geometry>
@@ -149,5 +149,5 @@
         </geometry>
         <xacro:material_abb_yellow />
-      </collision>
+      </collision>-->
     </link>
     <link name="${prefix}tool0"/>

File: ws_husky_abb/husky_abb_description/urdf/husky_abb.urdf.xacro (robot description, xacro)
@@ -6,5 +6,4 @@
   <xacro:include filename="$(find barrett_hand)/urdf/barrett.xacro"/>
   <xacro:include filename="$(find husky_abb_description)/urdf/kinect.xacro"/>
-  <xacro:include filename="$(find husky_abb_description)/urdf/hokuyo.xacro"/>
   <!-- Fix robot to Gazebo world
   <link name="world"/>-->
@@ -21,9 +20,3 @@
     <child link="barrett_base_link"/>
   </joint>
-  <joint name="husky_hokuyo_link" type="fixed">
-    <axis xyz="0 1 0" />
-    <origin xyz="0.38 0 -0.125" rpy="0 0 0"/>
-    <parent link="top_plate_link"/>
-    <child link="hokuyo_link"/>
-  </joint>
  </robot>
